File: pcb/solder/gear60_solder.kicad_pcb (KiCad board)
At the start: 2 copper layers, 284.2 x 93.7 mm, 185 parts, among them J1 TYPE-C-31-M-12, J3 Conn_01x05, U1 XC6206P332MR, U2 SRV05-4, U3 W25Q128JVSIQ, U4 RP2040, Y1 X322512MSB4SI

Commit message: Add files via upload
Parts:
- added MX31: MX_SW_solder, PCM_marbastlib-mx:SW_MX_1u, F.Cu at (288.1, 52.4)
- added MX46: MX_SW_solder, PCM_marbastlib-mx:SW_MX_1u, F.Cu at (266.7, 61.9)
- added MX80: MX_SW_solder, PCM_marbastlib-mx:SW_MX_1.25u, F.Cu at (73.8, 100.0)
- added MX81: MX_SW_solder, PCM_marbastlib-mx:SW_MX_1.25u, F.Cu at (50.0, 100.0)
- added MX82: MX_SW_solder, PCM_marbastlib-mx:SW_MX_1.25u, F.Cu at (26.2, 100.0)
- added MX83: MX_SW_solder, PCM_marbastlib-mx:SW_MX_1u, F.Cu at (145.3, 100.0)
- added MX84: MX_SW_solder, PCM_marbastlib-mx:SW_MX_1.25u, F.Cu at (216.7, 100.0)
- added MX85: MX_SW_solder, PCM_marbastlib-mx:SW_MX_1.25u, F.Cu at (288.1, 100.0)
- added MX86: MX_SW_solder, PCM_marbastlib-mx:SW_MX_1.25u, F.Cu at (264.3, 100.0)
- added S8: stb, PCM_marbastlib-mx:STAB_MX_P_6.25u, F.Cu at (145.3, 100.0)
- added S9: stb, PCM_marbastlib-mx:STAB_MX_ISO, F.Cu at (288.1, 52.4)
- moved D71 8.98 mm to (272.1, 103.2), turned to -90 degrees
- moved D30 5.99 mm to (293.5, 47.4)
- moved C12 4.67 mm to (134.9, 105.4)
- moved Y1 4.62 mm to (136.9, 103.6)
- moved R9 4.36 mm to (135.4, 101.8)
- moved C11 4.31 mm to (139.0, 105.3)
- moved C13 4.31 mm to (137.6, 85.9)
- moved C14 4.31 mm to (136.6, 85.9)
- moved C3 4.31 mm to (133.2, 87.2)
- moved C4 4.31 mm to (132.9, 101.3)
- moved C8 4.31 mm to (142.4, 89.9)
- moved R8 4.31 mm to (134.6, 84.5)
- moved C15 4.31 mm to (134.8, 100.4)
- moved C16 4.31 mm to (132.1, 87.2)
- moved R7 4.31 mm to (135.6, 84.5)
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Connections:
- U4 pad 11: unconnected-(U4-GPIO8-Pad11) -> COL8
- U4 pad 12: COL8 -> COL9
- U4 pad 13: COL9 -> COL10
- U4 pad 14: COL10 -> COL7
- U4 pad 15: COL7 -> unconnected-(U4-GPIO12-Pad15)
- U4 pad 6: ROW3 -> COL13
- U4 pad 7: ROW4 -> ROW3
- U4 pad 9: COL13 -> ROW4
Routing:
- net COL14: track 292.3 -> 319.9 mm
- net COL12: track 247.8 -> 260.9 mm
- net Net-(D67-A): track 15.8 -> 27.7 mm
- net Net-(D45-A): track 4.36 -> 16.3 mm
- net COL7: track 129.7 -> 141.3 mm
- net Net-(D71-A): track 15.9 -> 27.3 mm
- net Net-(D30-A): track 4.36 -> 15.7 mm
- net ROW1: track 336.7 -> 346.4 mm
- net COL10: track 179.2 -> 186.5 mm
- net COL8: track 107.1 -> 113.4 mm
- net ROW4: track 329.9 -> 324.1 mm, vias 4 -> 3
- net COL6: track 92.6 -> 87.5 mm
- net COL3: track 141.4 -> 136.6 mm
- net COL0: track 192.8 -> 188.0 mm
- net QSPI_SS: track 51.5 -> 56.1 mm
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
Commit message: Add files via upload
Parts:
- moved D45 11.9 mm to (269.8, 62.6)
Routing:
- net ROW2: track 345.0 -> 333.0 mm
