File: pcb/solder/gear60_solder.kicad_pcb (KiCad board)
At the start: 2 copper layers, 284.2 x 93.7 mm, 196 parts, among them J1 TYPE-C-31-M-12, J3 Conn_01x05, U1 XC6206P332MR, U2 SRV05-4, U3 W25Q128JVSIQ, U4 RP2040, Y1 X322512MSB4SI

Commit message: Add files via upload
Parts:
- moved D70 10.3 mm to (247.4, 103.7)
- moved D63 6.88 mm to (35.7, 103.7), turned to -90 degrees
- moved D69 3.08 mm to (222.8, 103.7)
- moved D71 1.74 mm to (270.5, 103.7)
- moved D72 1.48 mm to (278.4, 103.7)
- moved D64 0.79 mm to (46.6, 103.7)
Routing:
- net ROW4: track 324.1 -> 339.0 mm
- net GND: track 132.7 -> 123.7 mm, vias 27 -> 26
- net Net-(D69-A): track 6.74 -> 12.7 mm
- net COL5: track 126.9 -> 121.0 mm
- net Net-(D63-A): track 25.4 -> 19.7 mm
- net COL8: track 113.4 -> 110.5 mm
- net COL7: track 141.3 -> 139.3 mm
- net COL10: track 186.5 -> 184.5 mm
- net COL12: track 260.9 -> 259.0 mm
- net COL9: track 158.2 -> 156.2 mm
- net Net-(D71-A): track 27.3 -> 25.9 mm
- net COL11: track 208.4 -> 207.2 mm
- net COL2: track 178.1 -> 177.1 mm
- net COL4: track 125.7 -> 124.9 mm
- net Net-(D64-A): track 24.2 -> 25.0 mm
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
Commit message: Add files via upload
Parts:
- moved D67 9.05 mm to (171.2, 103.7)
- moved D2 8.95 mm to (50.6, 24.3), turned to -90 degrees
- moved D49 4.71 mm to (55.4, 81.5)
- moved D15 4.11 mm to (278.4, 26.7)
- moved D30 3.81 mm to (293.5, 43.6)
- moved D48 3.27 mm to (18.1, 81.5)
- moved D14 3.13 mm to (264.1, 24.5)
- moved D1 1.22 mm to (20.7, 24.3)
- moved D61 0.79 mm to (282.4, 81.5)
Routing:
- net COL14: track 319.9 -> 312.9 mm
- net ROW0: track 368.6 -> 361.9 mm
- net Net-(D48-A): track 64.8 -> 58.2 mm
- net Net-(D49-A): track 17.0 -> 11.5 mm
- net Net-(D15-A): track 19.9 -> 15.5 mm
- net Net-(D14-A): track 13.1 -> 10.0 mm
- net Net-(D30-A): track 15.7 -> 18.5 mm
- net ROW3: track 326.2 -> 323.8 mm
- net Net-(D2-A): track 9.42 -> 11.5 mm
- net ROW1: track 346.4 -> 347.9 mm
- net Net-(D67-A): track 27.7 -> 29.3 mm
- net Net-(D61-A): track 22.9 -> 21.5 mm
- net Net-(D1-A): track 4.36 -> 3.14 mm
- net Net-(D17-A): track 9.58 -> 8.41 mm
- net COL12: track 259.0 -> 258.2 mm

Commit message: Add files via upload
Parts:
- moved D15 0.79 mm to (278.4, 27.5)
