File: pcb/solder/gear60_solder.kicad_pcb (KiCad board)
At the start: 2 copper layers, 284.2 x 93.7 mm, 196 parts, among them J1 TYPE-C-31-M-12, J3 Conn_01x05, U1 XC6206P332MR, U2 SRV05-4, U3 W25Q128JVSIQ, U4 RP2040, Y1 X322512MSB4SI

Commit message: Add files via upload
Parts:
- moved D33 1.59 mm to (18.1, 62.4)
- moved D17 1.16 mm to (18.1, 43.5)
Routing:
- net Net-(D64-A): track 25.0 -> 35.2 mm
- net COL14: track 312.9 -> 319.1 mm
- net ROW2: track 333.0 -> 327.3 mm
- net Net-(D33-A): track 20.1 -> 16.1 mm
- net ROW4: track 338.8 -> 340.9 mm
- net +3V3: track 179.8 -> 177.7 mm
- net COL2: track 177.1 -> 175.4 mm
- net Net-(D17-A): track 8.41 -> 9.55 mm
- net ROW1: track 347.9 -> 349.0 mm
- net RESET: track 53.7 -> 52.9 mm
- net COL6: track 86.8 -> 86.1 mm
- net GND: track 123.7 -> 123.1 mm

Commit message: Add files via upload
Parts:
- moved D65 1.59 mm to (67.3, 103.7)
Routing:
- net COL10: track 184.5 -> 180.4 mm
- net ROW4: track 340.9 -> 336.9 mm
- net Net-(D48-A): track 58.2 -> 61.4 mm
- net Net-(D65-A): track 25.1 -> 22.4 mm
- net COL4: track 124.9 -> 124.3 mm

Commit message: Add files via upload
Routing:
- net COL12: track 258.5 -> 261.3 mm
- net COL5: track 120.6 -> 119.9 mm
Changed lines of the file:
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@@
   (segment (start 124.7775 40.3225) (end 124.7775 54.61) (width 0.2) (layer "F.Cu") (net 47))
   (segment (start 115.2525 30.7975) (end 124.7775 40.3225) (width 0.2) (layer "F.Cu") (net 47))
-  (segment (start 127.014289 67.20625) (end 130.307269 63.91327) (width 0.2) (layer "F.Cu") (net 47))
-  (segment (start 130.307269 63.91327) (end 130.307269 61.908603) (width 0.2) (layer "F.Cu") (net 47))
-  (segment (start 130.307269 61.908603) (end 129.54 61.141334) (width 0.2) (layer "F.Cu") (net 47))
+  (segment (start 120.015 78.4225) (end 120.015 71.955717) (width 0.2) (layer "F.Cu") (net 47))
+  (segment (start 120.015 83.9042) (end 112.87125 91.04795) (width 0.2) (layer "F.Cu") (net 47))
+  (segment (start 127.014289 67.20625) (end 129.54 64.680539) (width 0.2) (layer "F.Cu") (net 47))
+  (segment (start 129.54 64.680539) (end 129.54 59.3725) (width 0.2) (layer "F.Cu") (net 47))
+  (segment (start 120.015 78.4225) (end 120.015 83.9042) (width 0.2) (layer "F.Cu") (net 47))
+  (segment (start 124.7775 54.61) (end 129.54 59.3725) (width 0.2) (layer "F.Cu") (net 47))
   (segment (start 124.764467 67.20625) (end 127.014289 67.20625) (width 0.2) (layer "F.Cu") (net 47))
+  (segment (start 112.87125 91.04795) (end 112.87125 97.4725) (width 0.2) (layer "F.Cu") (net 47))
   (segment (start 120.015 71.955717) (end 124.764467 67.20625) (width 0.2) (layer "F.Cu") (net 47))
-  (segment (start 120.015 83.9042) (end 112.87125 91.04795) (width 0.2) (layer "F.Cu") (net 47))
-  (segment (start 120.015 78.4225) (end 120.015 83.9042) (width 0.2) (layer "F.Cu") (net 47))
-  (segment (start 120.015 78.4225) (end 120.015 71.955717) (width 0.2) (layer "F.Cu") (net 47))
-  (segment (start 124.7775 54.61) (end 129.54 59.3725) (width 0.2) (layer "F.Cu") (net 47))
-  (segment (start 112.87125 91.04795) (end 112.87125 97.4725) (width 0.2) (layer "F.Cu") (net 47))
-  (segment (start 129.54 61.141334) (end 129.54 59.3725) (width 0.2) (layer "F.Cu") (net 47))
   (segment (start 131.809538 97.909212) (end 133.188715 97.909212) (width 0.2) (layer "B.Cu") (net 47))
   (segment (start 134.123151 97.60891) (end 134.123151 96.727962) (width 0.2) (layer "B.Cu") (net 47))
@@
   (segment (start 136.452801 57.395301) (end 135.89 56.8325) (width 0.25) (layer "B.Cu") (net 58))
   (segment (start 263.675514 92.336323) (end 258.501177 92.336323) (width 0.2) (layer "F.Cu") (net 59))
-  (segment (start 243.84 59.3725) (end 243.84 61.066781) (width 0.2) (layer "F.Cu") (net 59))
   (segment (start 239.0775 40.3225) (end 239.0775 54.61) (width 0.2) (layer "F.Cu") (net 59))
   (segment (start 265.308946 90.702891) (end 263.675514 92.336323) (width 0.2) (layer "F.Cu") (net 59))
+  (segment (start 243.84 59.3725) (end 243.84 69.591964) (width 0.2) (layer "F.Cu") (net 59))
   (segment (start 265.308946 85.071446) (end 265.308946 90.702891) (width 0.2) (layer "F.Cu") (net 59))
-  (segment (start 260.9375 81.875126) (end 262.564874 83.5025) (width 0.2) (layer "F.Cu") (net 59))
   (segment (start 263.74 83.5025) (end 263.31875 83.5025) (width 0.2) (layer "F.Cu") (net 59))
-  (segment (start 260.9375 80.7) (end 260.9375 81.875126) (width 0.2) (layer "F.Cu") (net 59))
   (segment (start 239.0775 54.61) (end 243.84 59.3725) (width 0.2) (layer "F.Cu") (net 59))
   (segment (start 248.6025 21.2725) (end 248.6025 30.7975) (width 0.2) (layer "F.Cu") (net 59))
+  (segment (start 257.750536 83.5025) (end 263.31875 83.5025) (width 0.2) (layer "F.Cu") (net 59))
   (segment (start 248.6025 30.7975) (end 239.0775 40.3225) (width 0.2) (layer "F.Cu") (net 59))
-  (segment (start 243.84 61.066781) (end 244.519805 61.746586) (width 0.2) (layer "F.Cu") (net 59))
-  (segment (start 262.564874 83.5025) (end 263.31875 83.5025) (width 0.2) (layer "F.Cu") (net 59))
-  (segment (start 244.519805 64.282305) (end 260.9375 80.7) (width 0.2) (layer "F.Cu") (net 59))
+  (segment (start 243.84 69.591964) (end 257.750536 83.5025) (width 0.2) (layer "F.Cu") (net 59))
   (segment (start 268.12875 83.5025) (end 263.31875 83.5025) (width 0.2) (layer "F.Cu") (net 59))
   (segment (start 258.501177 92.336323) (end 253.365 97.4725) (width 0.2) (layer "F.Cu") (net 59))
-  (segment (start 244.519805 61.746586) (end 244.519805 64.282305) (width 0.2) (layer "F.Cu") (net 59))
   (segment (start 265.308946 85.071446) (end 263.74 83.5025) (width 0.2) (layer "F.Cu") (net 59))
   (segment (start 174.994929 104.057101) (end 215.508933 104.057101) (width 0.2) (layer "B.Cu") (net 59))

Commit message: Add files via upload
Connections:
- MX63 pad 1: Net-(D48-A) -> COL0
- MX73 pad 2: Net-(D48-A) -> COL0
- MX82 pad 1: Net-(D48-A) -> COL0
Routing:
- net COL0: track 188.0 -> 222.9 mm
- net Net-(D48-A): track 61.4 -> 30.7 mm
