File: pcb/solder/gear60_solder.kicad_sch (KiCad schematic)
At the start: 185 parts, among them J1 TYPE-C-31-M-12, J3 Conn_01x05, U1 XC6206P332MR, U2 SRV05-4, U3 W25Q128JVSIQ, U4 RP2040, Y1 X322512MSB4SI

Commit message: Add files via upload
Parts:
- added MX31, MX46, MX83: MX_SW_solder, PCM_marbastlib-mx:SW_MX_1u, symbol PCM_marbastlib-mx:MX_SW_HS
- added MX80, MX81, MX82, MX84, MX85, MX86: MX_SW_solder, PCM_marbastlib-mx:SW_MX_1.25u, symbol PCM_marbastlib-mx:MX_SW_HS
- added S8: stb, PCM_marbastlib-mx:STAB_MX_P_6.25u, symbol PCM_marbastlib-mx:MX_stab
- added S9: stb, PCM_marbastlib-mx:STAB_MX_ISO, symbol PCM_marbastlib-mx:MX_stab
Connections:
- net COL1: now also MX81.2
- net COL10: now also U4.13 (GPIO10), MX84.1; no longer U4.14 (GPIO11)
- net COL12: now also MX86.1
- net COL13: now also U4.6 (GPIO4); no longer U4.9 (GPIO7)
- net COL14: now also MX31.2, MX46.1, MX85.2
- net COL2: now also MX80.2
- net COL7: now also U4.14 (GPIO11), MX83.1; no longer U4.15 (GPIO12)
- net COL8: now also U4.11 (GPIO8); no longer U4.12 (GPIO9)
- net COL9: now also U4.12 (GPIO9); no longer U4.13 (GPIO10)
- net ROW3: now also U4.7 (GPIO5); no longer U4.6 (GPIO4)
- net ROW4: now also U4.9 (GPIO7); no longer U4.7 (GPIO5)
- net at D48.2 (A), MX47.2, MX48.2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: now also MX82.1
- net at D65.2 (A), MX65.2, MX75.1: now also MX80.1
- net at D71.2 (A), MX71.2, MX78.1: now also MX86.2
- net at D69.2 (A), MX69.2: now also MX84.2
- net at D45.2 (A), MX45.2: now also MX46.2
- net at D64.2 (A), MX64.2, MX74.1: now also MX81.1
- net at D30.2 (A), MX30.2: now also MX31.1
- net at D72.2 (A), MX72.2, MX79.1: now also MX85.1
- net at D63.2 (A), MX63.2, MX73.1: now also MX82.2
- net at D67.2 (A), MX67.1, MX76.2: now also MX83.2
Other:
- moved on the sheet: S3

Commit message: Add files via upload
Connections:
- net COL0: now also MX63.1, MX73.2, MX82.1
- net at D48.2 (A), MX47.2, MX48.2: no longer MX63.1, MX73.2, MX82.1
Changed lines of the file:
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@@
   (junction (at 245.11 128.27) (diameter 0) (color 0 0 0 0)
   )
+  (junction (at 245.11 121.92) (diameter 0) (color 0 0 0 0)
+  )
   (junction (at 417.83 95.25) (diameter 0) (color 0 0 0 0)
   )
@@
   (junction (at 281.94 142.24) (diameter 0) (color 0 0 0 0)
   )
-  (junction (at 240.03 121.92) (diameter 0) (color 0 0 0 0)
-  )
   (junction (at 452.12 80.01) (diameter 0) (color 0 0 0 0)
-  )
-  (junction (at 245.11 121.92) (diameter 0) (color 0 0 0 0)
   )
   (junction (at 115.57 182.88) (diameter 0) (color 0 0 0 0)
@@
     (stroke (width 0) (type default))
   )
-  (wire (pts (xy 240.03 121.92) (xy 245.11 121.92))
-    (stroke (width 0) (type default))
-  )
   (wire (pts (xy 245.11 86.36) (xy 260.35 86.36))
     (stroke (width 0) (type default))
@@
     (stroke (width 0) (type default))
   )
-  (wire (pts (xy 240.03 121.92) (xy 240.03 137.16))
+  (wire (pts (xy 240.03 116.84) (xy 240.03 137.16))
     (stroke (width 0) (type default))
   )
@@
     (stroke (width 0) (type default))
   )
-  (wire (pts (xy 237.49 121.92) (xy 240.03 121.92))
-    (stroke (width 0) (type default))
-  )
   (wire (pts (xy 407.67 106.68) (xy 422.91 106.68))
     (stroke (width 0) (type default))
@@
     (stroke (width 0) (type default))
   )
+  (wire (pts (xy 237.49 121.92) (xy 245.11 121.92))
+    (stroke (width 0) (type default))
+  )

Commit message: Add files via upload
Parts:
- removed J3: Conn_01x05, Connector_PinHeader_2.54mm:PinHeader_1x05_P2.54mm_Vertical, symbol Connector_Generic:Conn_01x05
- added MX87, MX88, MX89: MX_SW_solder, PCM_marbastlib-mx:SW_MX_1u, symbol PCM_marbastlib-mx:MX_SW_HS
Connections:
- net COL5: now also MX66.2, MX87.1; no longer MX66.1
- net COL7: now also MX67.1, MX88.2; no longer MX67.2
- net COL9: now also MX89.2
- net at D66.2 (A): now also MX66.1, MX87.2; no longer MX66.2
- net at D67.2 (A), MX76.2, MX83.2: now also MX67.2, MX88.1; no longer MX67.1
- net at D68.2 (A), MX68.2: now also MX89.1
Other:
- note removed: "SWD"
- moved on the sheet: MX66, MX67, MX68, S2, S4

Commit message: Add files via upload
Parts:
- C5: value 10u -> 100n; footprint Capacitor_SMD:C_0603_1608Metric -> Capacitor_SMD:C_0402_1005Metric
Changed lines of the file:
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@@
+    )
+  )
+  (symbol (lib_id "Device:C_Small") (at 118.11 146.05 0) (unit 1)
+    (in_bom yes) (on_board yes) (dnp no) (fields_autoplaced)
+    (property "Reference" "C5" (at 120.65 144.7863 0)
+      (effects (font (size 1.27 1.27)) (justify left))
+    )
+    (property "Value" "100n" (at 120.65 147.3263 0)
+      (effects (font (size 1.27 1.27)) (justify left))
+    )
+    (property "Footprint" "Capacitor_SMD:C_0402_1005Metric" (at 118.11 146.05 0)
+      (effects (font (size 1.27 1.27)) hide)
+    )
+    (property "Datasheet" "~" (at 118.11 146.05 0)
+      (effects (font (size 1.27 1.27)) hide)
+    )
+    (pin "1")
+    (pin "2")
+    (instances
+      (project "gear60_solder"
+        (path "/b7ecd40f-fbd1-4363-aa36-fbfbff6aee59"
+          (reference "C5") (unit 1)
+        )
+      )
     )
   )
@@
         )
       )
-    )
-  )
-  (symbol (lib_id "Device:C_Small") (at 118.11 146.05 0) (unit 1)
-    (in_bom yes) (on_board yes) (dnp no) (fields_autoplaced)
-    (property "Reference" "C5" (at 120.65 144.7863 0)
-      (effects (font (size 1.27 1.27)) (justify left))
-    )
-    (property "Value" "10u" (at 120.65 147.3263 0)
-      (effects (font (size 1.27 1.27)) (justify left))
-    )
-    (property "Footprint" "Capacitor_SMD:C_0603_1608Metric" (at 118.11 146.05 0)
-      (effects (font (size 1.27 1.27)) hide)
-    )
-    (property "Datasheet" "~" (at 118.11 146.05 0)
-      (effects (font (size 1.27 1.27)) hide)
-    )
-    (pin "1")
-    (pin "2")
-    (instances
-      (project "gear60_solder"
-        (path "/b7ecd40f-fbd1-4363-aa36-fbfbff6aee59"
-          (reference "C5") (unit 1)
-        )
-      )
