File: pcb/solder_rp2040zero/gear60_solder_rp2040zero.kicad_pcb (KiCad board)
At the start: 2 copper layers, 284.2 x 93.7 mm, 163 parts, among them U1 rp2040-zero

Commit message: Add files via upload
Connections:
- U1 pad 22: unconnected-(U1-GND-Pad22) -> GND
Routing:
- net GND: track 0.00 -> 1.22 mm, vias 0 -> 1
- added copper zone on B.Cu, net GND
- added copper zone on F.Cu, net GND
