File: pcb/solder_rp2040zero/gear60_solder_rp2040zero.kicad_sch (KiCad schematic)
At the start: 163 parts, among them U1 rp2040-zero

Commit message: Add files via upload
Connections:
- net GND: now reaches U1.22 (GND)
- no-connect marks 0 -> 2
